File: kicad/ochrana-krby-lcd-teplotni-senzor/ochrana-krby-lcd-teplotni-senzor.sch (KiCad schematic (older format))
At the start: 7 parts, among them J1 Screw_Terminal_01x03, P1 1x2_pins_header_rl, Q1 BSS138P

Commit message: Adding of information and small changes. Remove main.pdf is too large.
Parts:
- D6: value undir_transil -> ESD9L5.0ST5G
Changed lines of the file:
@@
 P 4700 3100
 F 0 "D6" H 4794 3146 50  0000 L CNN
-F 1 "undir_transil" H 4794 3055 50  0000 L CNN
+F 1 "ESD9L5.0ST5G" H 4794 3055 50  0000 L CNN
 F 2 "diodes_smd_rl:sod_323_rl" H 4700 3100 50  0001 C CNN
 F 3 "" H 4700 3100 50  0001 C CNN
@@
 U 1 1 5FE1040C
 P 4100 3000
-F 0 "D1" H 4100 3335 50  0000 C CNN
-F 1 "DS9503" H 4100 3244 50  0000 C CNN
+F 0 "D1" H 4100 3250 50  0000 C CNN
+F 1 "DS9503" H 4100 2750 50  0000 C CNN
 F 2 "" H 4100 3000 50  0001 C CNN
 F 3 "" H 4100 3000 50  0001 C CNN

Commit message: Adding of new parts and modify old parts.
Parts:
- D1: symbol diodes_rl:DS9503_eu_rl -> ochrana-krby-lcd-teplotni-senzor-rescue:DS9503_eu_rl-diodes_rl
- D6: symbol diodes_rl:undir_transil -> ochrana-krby-lcd-teplotni-senzor-rescue:undir_transil-diodes_rl
- P1: symbol connectors_rl:1x2_pins_header_rl -> ochrana-krby-lcd-teplotni-senzor-rescue:1x2_pins_header_rl-connectors_rl
Other:
- note added: "Modrá LED"
- note added: "Oranžová LED"
- note added: "Vstupní řídicí signál"
- note added: "Červená LED"
- note removed: "blue"
- note removed: "input\ncontrol\nsignal"
- note removed: "orange"
- note removed: "red"
- note removed: "red LED"
Changed lines of the file:
@@
 $EndComp
 $Comp
-L diodes_rl:undir_transil D6
+L ochrana-krby-lcd-teplotni-senzor-rescue:undir_transil-diodes_rl D6
 U 1 1 5E8F4FAB
 P 4700 3100
@@
 	5850 2900 5500 2900
 $Comp
-L connectors_rl:1x2_pins_header_rl P1
+L ochrana-krby-lcd-teplotni-senzor-rescue:1x2_pins_header_rl-connectors_rl P1
 U 1 1 5F44F2DA
 P 6300 2400
@@
 Connection ~ 5500 3300
 Text Notes 6250 2250 0    50   ~ 0
-red LED
-Text Notes 3000 2850 0    50   ~ 0
-input\ncontrol\nsignal
-Text Notes 2550 3150 0    50   ~ 0
-blue
-Text Notes 2460 3030 0    50   ~ 0
-orange
-Text Notes 2600 2900 0    50   ~ 0
-red
+Červená LED
+Text Notes 2950 2800 0    50   ~ 0
+Vstupní řídicí signál
+Text Notes 2300 3200 0    50   ~ 0
+Modrá LED
+Text Notes 2200 3050 0    50   ~ 0
+Oranžová LED
+Text Notes 2250 2900 0    50   ~ 0
+Červená LED
 Wire Wire Line
 	3000 2900 3800 2900
@@
 $EndComp
 $Comp
-L diodes_rl:DS9503_eu_rl D1
+L ochrana-krby-lcd-teplotni-senzor-rescue:DS9503_eu_rl-diodes_rl D1
 U 1 1 5FE1040C
 P 4100 3000
