File: kicad/ochrana-napajeni-3_3-v/ochrana-napajeni-3_3-v.sch (KiCad schematic (older format))
At the start: 3 parts, among them J6 1x2_screw_term_block

Commit message: Adding of information and small changes. Remove main.pdf is too large.
Parts:
- D17: value undir_transil -> SM2T3V3A
- F1: value Polyfuse -> RXEF005
Changed lines of the file:
@@
 P 4950 2650
 F 0 "F1" V 4725 2650 50  0000 C CNN
-F 1 "Polyfuse" V 4816 2650 50  0000 C CNN
+F 1 "RXEF005" V 4816 2650 50  0000 C CNN
 F 2 "fuses_tht_rl:fuse_littelfuse_rxef_series" H 5000 2450 50  0001 L CNN
 F 3 "~" H 4950 2650 50  0001 C CNN
@@
 P 4500 2900
 F 0 "D17" H 4594 2946 50  0000 L CNN
-F 1 "undir_transil" H 4594 2855 50  0000 L CNN
+F 1 "SM2T3V3A" H 4594 2855 50  0000 L CNN
 F 2 "diodes_smd_rl:do_216aa" H 4500 2900 50  0001 C CNN
 F 3 "" H 4500 2900 50  0001 C CNN

Commit message: Adding of new parts and modify old parts.
Parts:
- J6: symbol connectors_rl:1x2_screw_term_block -> ochrana-napajeni-3_3-v-rescue:1x2_screw_term_block-connectors_rl
Other:
- note added: "Vstup 3,3 V z RPI"
- note added: "Výstup 3,3 V"
- note removed: "input voltage\nfrom RPI +3,3 V"
- note removed: "output \nvoltage\n+3,3 V"
Changed lines of the file:
@@
 	4350 2400 4350 2650
 $Comp
-L connectors_rl:1x2_screw_term_block J6
+L ochrana-napajeni-3_3-v-rescue:1x2_screw_term_block-connectors_rl J6
 U 1 1 5F2AB78D
 P 5200 2250
@@
 $EndComp
 Text Notes 5000 2150 0    50   ~ 0
-input voltage\nfrom RPI +3,3 V
-Text Notes 4000 2700 0    50   ~ 0
-output \nvoltage\n+3,3 V
+Vstup 3,3 V z RPI
+Text Notes 3800 2700 0    50   ~ 0
+Výstup 3,3 V
 $EndSCHEMATC
