File: kicad/max31850k-1-wire-prevodnik-termoclanku/max31850k-1-wire-prevodnik-termoclanku.sch (KiCad schematic (older format))
At the start: 23 parts, among them J1 DG390-5.0, J2 1x4_pins_grove_rl, Q1 2N7002, U1 XC6206P332MR-G, U2 MAX31850K

Commit message: Adding of new parts and modify old parts.
Parts:
- C1, C2, C3, C4, C5, C6, C7, C8: symbol passive_components_rl:capacitor_rl -> max31850k-1-wire-prevodnik-termoclanku-rescue:capacitor_rl-passive_components_rl
- J1: symbol connectors_rl:DG390-5.0_rl -> max31850k-1-wire-prevodnik-termoclanku-rescue:DG390-5.0_rl-connectors_rl
- J2: symbol connectors_rl:1x4_pins_grove_rl -> max31850k-1-wire-prevodnik-termoclanku-rescue:1x4_pins_grove_rl-connectors_rl
- L1, L2: symbol passive_components_rl:inductor_rl -> max31850k-1-wire-prevodnik-termoclanku-rescue:inductor_rl-passive_components_rl
- U2: symbol thermocouples_rl:MAX31850K_rl -> max31850k-1-wire-prevodnik-termoclanku-rescue:MAX31850K_rl-thermocouples_rl
Other:
- note added: "Adresace"
- note added: "LDO"
- note added: "Převodník log. úrovně"
- note added: "Termočlánek"
- note added: "Vstup/výstup"
- note removed: "adresses"
- note removed: "input/output"
- note removed: "level shifter"
- note removed: "power supply"
- note removed: "thermocouple"
Changed lines of the file:
@@
 $EndDescr
 $Comp
-L thermocouples_rl:MAX31850K_rl U2
+L max31850k-1-wire-prevodnik-termoclanku-rescue:MAX31850K_rl-thermocouples_rl U2
 U 1 1 5FE095CF
 P 4850 3450
@@
 	4850 3800 4850 4100
 $Comp
-L passive_components_rl:capacitor_rl C5
+L max31850k-1-wire-prevodnik-termoclanku-rescue:capacitor_rl-passive_components_rl C5
 U 1 1 5FE0D623
 P 3400 3000
@@
 $EndComp
 $Comp
-L passive_components_rl:capacitor_rl C6
+L max31850k-1-wire-prevodnik-termoclanku-rescue:capacitor_rl-passive_components_rl C6
 U 1 1 5FE0E09B
 P 3400 3400
@@
 $EndComp
 $Comp
-L passive_components_rl:capacitor_rl C7
+L max31850k-1-wire-prevodnik-termoclanku-rescue:capacitor_rl-passive_components_rl C7
 U 1 1 5FE0E717
 P 3400 3800
@@
 	2650 3200 3400 3200
 $Comp
-L passive_components_rl:inductor_rl L1
+L max31850k-1-wire-prevodnik-termoclanku-rescue:inductor_rl-passive_components_rl L1
 U 1 1 5FE1AEF9
 P 2150 3200
@@
 $EndComp
 $Comp
-L passive_components_rl:inductor_rl L2
+L max31850k-1-wire-prevodnik-termoclanku-rescue:inductor_rl-passive_components_rl L2
 U 1 1 5FE1BFAF
 P 2150 3600
@@
 Connection ~ 2650 3200
 $Comp
-L connectors_rl:DG390-5.0_rl J1
+L max31850k-1-wire-prevodnik-termoclanku-rescue:DG390-5.0_rl-connectors_rl J1
 U 1 1 5FE1FE3F
 P 1600 3400
@@
 	2550 4100 2550 4050
 $Comp
-L passive_components_rl:capacitor_rl C8
+L max31850k-1-wire-prevodnik-termoclanku-rescue:capacitor_rl-passive_components_rl C8
 U 1 1 5FE31334
 P 4050 3800
@@
 dq
 $Comp
-L passive_components_rl:capacitor_rl C2
+L max31850k-1-wire-prevodnik-termoclanku-rescue:capacitor_rl-passive_components_rl C2
 U 1 1 5FE387C4
 P 2100 2200
@@
 $EndComp
 $Comp
-L passive_components_rl:capacitor_rl C1
+L max31850k-1-wire-prevodnik-termoclanku-rescue:capacitor_rl-passive_components_rl C1
 U 1 1 5FE399C9
 P 1650 2200
@@
 	2100 2000 2250 2000
 $Comp
-L passive_components_rl:capacitor_rl C3
+L max31850k-1-wire-prevodnik-termoclanku-rescue:capacitor_rl-passive_components_rl C3
 U 1 1 5FE3C738
 P 3000 2200
@@
 $EndComp
 $Comp
-L passive_components_rl:capacitor_rl C4
+L max31850k-1-wire-prevodnik-termoclanku-rescue:capacitor_rl-passive_components_rl C4
 U 1 1 5FE3D2ED
 P 3400 2200
@@
 	1900 4300 1900 4250
 $Comp
-L connectors_rl:1x4_pins_grove_rl J2
+L max31850k-1-wire-prevodnik-termoclanku-rescue:1x4_pins_grove_rl-connectors_rl J2
 U 1 1 5FEA3614
 P 6450 3500
@@
 ad0
 Text Notes 1400 3700 0    50   ~ 0
-thermocouple
+Termočlánek
 Text Notes 6150 3900 0    50   ~ 0
-input/output
+Vstup/výstup
 Text Notes 2850 4550 0    50   ~ 0
-adresses
-$Comp
-L power_rl:+3,3V #PWR1
+Adresace
+$Comp
+L max31850k-1-wire-prevodnik-termoclanku-rescue:+3,3V-power_rl #PWR1
 U 1 1 5FEC5542
 P 3400 1950
@@
 	3400 2000 3800 2000
 $Comp
-L power_rl:+3,3V #PWR3
+L max31850k-1-wire-prevodnik-termoclanku-rescue:+3,3V-power_rl #PWR3
 U 1 1 5FECC748
 P 4500 1950
@@
 $EndComp
 $Comp
-L power_rl:+3,3V #PWR4
+L max31850k-1-wire-prevodnik-termoclanku-rescue:+3,3V-power_rl #PWR4
 U 1 1 5FECD33A
 P 1900 4250
@@
 $EndComp
 $Comp
-L power_rl:+3,3V #PWR2
+L max31850k-1-wire-prevodnik-termoclanku-rescue:+3,3V-power_rl #PWR2
 U 1 1 5FECFF7B
 P 4050 3100
@@
 	1    0    0    -1
 $EndComp
-Text Notes 2300 1700 0    50   ~ 0
-power supply
+Text Notes 2500 1650 0    50   ~ 0
+LDO
 Text Notes 4750 1750 0    50   ~ 0
-level shifter
+Převodník log. úrovně
 $Comp
 L Device:R R3

Commit message: Adding of HW parts and small changes.
Parts:
- J2: value 1x4_pins_grove_rl -> 1x4_pins_grove
Changed lines of the file:
@@
 P 6450 3500
 F 0 "J2" V 6150 3400 50  0000 L CNN
-F 1 "1x4_pins_grove_rl" V 6700 3150 50  0000 L CNN
+F 1 "1x4_pins_grove" V 6700 3150 50  0000 L CNN
 F 2 "" H 6350 3500 50  0001 C CNN
 F 3 "" H 6350 3500 50  0001 C CNN
