File: kicad/pca9615-i2-sbernice/pca9615-i2-sbernice.sch (KiCad schematic (older format))
At the start: 18 parts, among them J1 rj45_rl, J2 1x2_screw_term_block, P1 1x5_pins_header_rl, U1 PCA9615

Commit message: Adding of HW parts and small changes.
Parts:
- C1, C2, C3, C4: symbol passive_components_rl:capacitor_rl -> pca9615-i2-sbernice-rescue:capacitor_rl-passive_components_rl
- J1: value rj45_rl -> rj45; symbol connectors_rl:rj45_rl -> pca9615-i2-sbernice-rescue:rj45_rl-connectors_rl
- J2: symbol connectors_rl:1x2_screw_term_block -> pca9615-i2-sbernice-rescue:1x2_screw_term_block-connectors_rl
- P1: value 1x5_pins_header_rl -> 1x5_pins_header; symbol connectors_rl:1x5_pins_header_rl -> pca9615-i2-sbernice-rescue:1x5_pins_header_rl-connectors_rl
- R1, R3: value 390 -> 390R; symbol Device:R -> passive_component_rl:resistor_eu
- R2, R5: value 100 -> 100R
- R4, R6: value 390 -> 390R
- R7, R8: symbol passive_components_rl:resistor_rl -> passive_component_rl:resistor_eu
- U1: symbol interface_i2c_rl:PCA9615_RL -> pca9615-i2-sbernice-rescue:PCA9615_RL-interface_i2c_rl
Connections:
- net GND: now also R3.1; no longer R3.2
- net VDD_A: now also R1.2; no longer R1.1
- net dsclm: now also R3.2; no longer R3.1
- net dsclp: now also R1.1; no longer R1.2
Changed lines of the file:
@@
 $EndDescr
 $Comp
-L interface_i2c_rl:PCA9615_RL U1
+L pca9615-i2-sbernice-rescue:PCA9615_RL-interface_i2c_rl U1
 U 1 1 5FDFA46C
 P 3350 2200
@@
 $EndComp
 $Comp
-L connectors_rl:rj45_rl J1
+L pca9615-i2-sbernice-rescue:rj45_rl-connectors_rl J1
 U 1 1 5FDFAE21
 P 7100 3000
 F 0 "J1" H 7150 2450 50  0000 R CNN
-F 1 "rj45_rl" H 7200 2550 50  0000 R CNN
+F 1 "rj45" H 7200 2550 50  0000 R CNN
 F 2 "" H 7100 3000 50  0001 C CNN
 F 3 "" H 7100 3000 50  0001 C CNN
@@
 dsdam
 $Comp
-L passive_components_rl:capacitor_rl C1
+L pca9615-i2-sbernice-rescue:capacitor_rl-passive_components_rl C1
 U 1 1 5FE0FF60
 P 4300 3800
@@
 $EndComp
 $Comp
-L passive_components_rl:capacitor_rl C2
+L pca9615-i2-sbernice-rescue:capacitor_rl-passive_components_rl C2
 U 1 1 5FE10909
 P 4850 3800
@@
 $EndComp
 $Comp
-L passive_components_rl:capacitor_rl C3
+L pca9615-i2-sbernice-rescue:capacitor_rl-passive_components_rl C3
 U 1 1 5FE1103A
 P 5400 3800
@@
 $EndComp
 $Comp
-L passive_components_rl:capacitor_rl C4
+L pca9615-i2-sbernice-rescue:capacitor_rl-passive_components_rl C4
 U 1 1 5FE11A8F
 P 5950 3800
@@
 	3050 1300 3350 1300
 $Comp
-L connectors_rl:1x2_screw_term_block J2
+L pca9615-i2-sbernice-rescue:1x2_screw_term_block-connectors_rl J2
 U 1 1 5FE4995C
 P 4550 1200
@@
 	4200 1450 4200 1250
 $Comp
-L connectors_rl:1x5_pins_header_rl P1
+L pca9615-i2-sbernice-rescue:1x5_pins_header_rl-connectors_rl P1
 U 1 1 5FE5EC7F
 P 3000 3550
 F 0 "P1" V 3425 3481 50  0000 C CNN
-F 1 "1x5_pins_header_rl" V 3334 3481 50  0000 C CNN
+F 1 "1x5_pins_header" V 3334 3481 50  0000 C CNN
 F 2 "" H 3000 3550 50  0001 C CNN
 F 3 "" H 3000 3550 50  0001 C CNN
@@
 $EndComp
 $Comp
-L passive_components_rl:resistor_rl R7
+L passive_component_rl:resistor_eu R7
 U 1 1 5FE6FFB2
 P 5050 5050
@@
 $EndComp
 $Comp
-L passive_components_rl:resistor_rl R8
+L passive_component_rl:resistor_eu R8
 U 1 1 5FE7108F
 P 5750 5050
@@
 	5400 4600 5400 4550
 $Comp
-L Device:R R1
+L passive_component_rl:resistor_eu R1
 U 1 1 5FE0C9DD
 P 5000 2000
-F 0 "R1" H 5070 2046 50  0000 L CNN
-F 1 "390" H 5070 1955 50  0000 L CNN
+F 0 "R1" V 5050 1850 50  0000 L CNN
+F 1 "390R" V 4950 1750 50  0000 L CNN
 F 2 "" V 4930 2000 50  0001 C CNN
 F 3 "~" H 5000 2000 50  0001 C CNN
 	1    5000 2000
-	1    0    0    -1
+	0    -1   -1   0
 $EndComp
 $Comp
@@
 P 5000 2400
 F 0 "R2" H 5070 2446 50  0000 L CNN
-F 1 "100" H 5070 2355 50  0000 L CNN
+F 1 "100R" H 5070 2355 50  0000 L CNN
 F 2 "" V 4930 2400 50  0001 C CNN
 F 3 "~" H 5000 2400 50  0001 C CNN
@@
 $EndComp
 $Comp
-L Device:R R3
+L passive_component_rl:resistor_eu R3
 U 1 1 5FE0D4F7
 P 5000 2800
-F 0 "R3" H 5070 2846 50  0000 L CNN
-F 1 "390" H 5070 2755 50  0000 L CNN
+F 0 "R3" V 5050 2650 50  0000 L CNN
+F 1 "390R" V 4950 2550 50  0000 L CNN
 F 2 "" V 4930 2800 50  0001 C CNN
 F 3 "~" H 5000 2800 50  0001 C CNN
 	1    5000 2800
-	1    0    0    -1
+	0    -1   -1   0
 $EndComp
 $Comp
@@
 P 5950 2000
 F 0 "R4" H 6020 2046 50  0000 L CNN
-F 1 "390" H 6020 1955 50  0000 L CNN
+F 1 "390R" H 6020 1955 50  0000 L CNN
 F 2 "" V 5880 2000 50  0001 C CNN
 F 3 "~" H 5950 2000 50  0001 C CNN
@@
 P 5950 2400
 F 0 "R5" H 6020 2446 50  0000 L CNN
-F 1 "100" H 6020 2355 50  0000 L CNN
+F 1 "100R" H 6020 2355 50  0000 L CNN
 F 2 "" V 5880 2400 50  0001 C CNN
 F 3 "~" H 5950 2400 50  0001 C CNN
@@
 P 5950 2800
 F 0 "R6" H 6020 2846 50  0000 L CNN
-F 1 "390" H 6020 2755 50  0000 L CNN
+F 1 "390R" H 6020 2755 50  0000 L CNN
 F 2 "" V 5880 2800 50  0001 C CNN
 F 3 "~" H 5950 2800 50  0001 C CNN
