File: kicad/rele-modul-jeden-kanal/rele-modul-jeden-kanal.sch (KiCad schematic (older format))
At the start: 10 parts, among them J1 Screw_Terminal_01x03, K1 srd-05vdc-sl-c, P1 1x6_pins_header, P2 1x2_pins_header, Q1 BC547A, U1 817C

Commit message: Adding of new parts and modify old parts.
Parts:
- D1: symbol diodes_rl:LED -> rele-modul-jeden-kanal-rescue:LED-diodes_rl
- P1: symbol connectors_rl:1x6_pins_header_rl -> rele-modul-jeden-kanal-rescue:1x6_pins_header_rl-connectors_rl
- P2: symbol connectors_rl:1x2_pins_header_rl -> rele-modul-jeden-kanal-rescue:1x2_pins_header_rl-connectors_rl
Other:
- note added: "Vstupní\nřídicí\nsignál"
- note added: "Zátěž"
- note removed: "input\ncontrol\nsignal"
- note removed: "power supply"
Changed lines of the file:
@@
 $EndComp
 $Comp
-L connectors_rl:1x6_pins_header_rl P1
+L rele-modul-jeden-kanal-rescue:1x6_pins_header_rl-connectors_rl P1
 U 1 1 5FE617FF
 P 1700 2700
@@
 $EndComp
 $Comp
-L connectors_rl:1x2_pins_header_rl P2
+L rele-modul-jeden-kanal-rescue:1x2_pins_header_rl-connectors_rl P2
 U 1 1 5FE638DA
 P 3150 1950
@@
 	3100 2100 3100 2200
 $Comp
-L diodes_rl:LED D1
+L rele-modul-jeden-kanal-rescue:LED-diodes_rl D1
 U 1 1 5FE6A2E7
 P 2500 3250
@@
 Text Label 2250 3250 2    50   ~ 0
 in1
-Text Notes 1700 2100 0    50   ~ 0
-input\ncontrol\nsignal
+Text Notes 1700 2050 0    50   ~ 0
+Vstupní\nřídicí\nsignál
 $Comp
 L power:+5V #PWR0103
@@
 $EndComp
 $Comp
-L power_rl:+3,3V #PWR2
+L rele-modul-jeden-kanal-rescue:+3,3V-power_rl #PWR2
 U 1 1 5FE7C30E
 P 2700 2100
@@
 $EndComp
 $Comp
-L power_rl:+3,3V #PWR1
+L rele-modul-jeden-kanal-rescue:+3,3V-power_rl #PWR1
 U 1 1 5FE7B7FD
 P 2000 2350
@@
 Wire Wire Line
 	3900 2200 4150 2200
-Text Notes 2950 1900 0    50   ~ 0
-power supply
+Text Notes 5800 2200 0    50   ~ 0
+Zátěž
 $EndSCHEMATC

Commit message: Adding of HW parts and small changes.
Parts:
- D1: value red LED -> Červená LED
- J1: value Screw_Terminal_01x03 -> 1x3_screw_term_block; symbol Connector:Screw_Terminal_01x03 -> connector_rl:1x3_screw_term_block
- R2: value 510 -> 510R
Changed lines of the file:
@@
 $EndDescr
 $Comp
-L Connector:Screw_Terminal_01x03 J1
+L connector_rl:1x3_screw_term_block J1
 U 1 1 5FE602A7
 P 5900 2550
 F 0 "J1" H 5850 2750 50  0000 L CNN
-F 1 "Screw_Terminal_01x03" V 5900 1500 50  0000 L CNN
+F 1 "1x3_screw_term_block" V 5900 1500 50  0000 L CNN
 F 2 "" H 5900 2550 50  0001 C CNN
 F 3 "~" H 5900 2550 50  0001 C CNN
@@
 P 3600 3250
 F 0 "R2" V 3500 3250 50  0000 C CNN
-F 1 "510" V 3700 3250 50  0000 C CNN
+F 1 "510R" V 3700 3250 50  0000 C CNN
 F 2 "" V 3530 3250 50  0001 C CNN
 F 3 "~" H 3600 3250 50  0001 C CNN
@@
 P 2500 3250
 F 0 "D1" H 2493 3467 50  0000 C CNN
-F 1 "red LED" H 2493 3376 50  0000 C CNN
+F 1 "Červená LED" H 2493 3376 50  0000 C CNN
 F 2 "" H 2500 3250 50  0001 C CNN
 F 3 "~" H 2500 3250 50  0001 C CNN
