File: kicad/ochrana-napajeni-1-wire/ochrana-napajeni-1-wire.sch (KiCad schematic (older format))
At the start: 13 parts, among them J1 1x2_screw_term_block, P3 1x2_pins_header_rl, U1 TPS26600

Commit message: Adding of new parts and modify old parts.
Parts:
- C1, C2, C3: symbol passive_components_rl:capacitor_rl -> ochrana-napajeni-1-wire-rescue:capacitor_rl-passive_components_rl
- J1: symbol connectors_rl:1x2_screw_term_block -> ochrana-napajeni-1-wire-rescue:1x2_screw_term_block-connectors_rl
- P3: symbol connectors_rl:1x2_pins_header_rl -> ochrana-napajeni-1-wire-rescue:1x2_pins_header_rl-connectors_rl
- R17: symbol passive_components_rl:resisitor_variable_eu_rl -> ochrana-napajeni-1-wire-rescue:resisitor_variable_eu_rl-passive_components_rl
Connections:
- net at U1.8 (RTN): now also C2.2, R12.2, R18.2
Other:
- note added: "Vstup 5 V"
- note added: "Výstup 5 V"
- note added: "Červená LED"
- note removed: "input\nvoltage +5 V"
- note removed: "max. limitation\nI=2,21 A"
- note removed: "output\nvoltage +5 V"
- note removed: "red LED"
Changed lines of the file:
@@
 $EndComp
 $Comp
-L connectors_rl:1x2_screw_term_block J1
+L ochrana-napajeni-1-wire-rescue:1x2_screw_term_block-connectors_rl J1
 U 1 1 5E7774D7
 P 5150 2000
@@
 	5750 3400 6100 3400
 $Comp
-L passive_components_rl:capacitor_rl C1
+L ochrana-napajeni-1-wire-rescue:capacitor_rl-passive_components_rl C1
 U 1 1 5F1AD2F7
 P 4300 2700
@@
 Connection ~ 4550 2900
 $Comp
-L passive_components_rl:capacitor_rl C3
+L ochrana-napajeni-1-wire-rescue:capacitor_rl-passive_components_rl C3
 U 1 1 5F1DD9A0
 P 7550 3100
@@
 	6050 2900 7050 2900
 $Comp
-L passive_components_rl:capacitor_rl C2
+L ochrana-napajeni-1-wire-rescue:capacitor_rl-passive_components_rl C2
 U 1 1 5F24E72A
 P 6650 3850
@@
 	6950 3100 5750 3100
 $Comp
-L connectors_rl:1x2_pins_header_rl P3
+L ochrana-napajeni-1-wire-rescue:1x2_pins_header_rl-connectors_rl P3
 U 1 1 5F29F6AB
 P 7000 3500
@@
 Wire Wire Line
 	7050 3300 7050 3350
-Text Notes 7100 3400 0    50   ~ 0
-red LED
+Text Notes 7000 3750 0    50   ~ 0
+Červená LED
 Wire Wire Line
 	6100 3400 6100 3650
@@
 Wire Wire Line
 	7100 2900 7450 2900
-Text Notes 5400 4400 0    50   ~ 0
-max. limitation\nI=2,21 A
-Text Notes 5300 4150 0    50   ~ 0
+Text Notes 5300 4250 0    50   ~ 0
 max. I = 0,073 A\n114,64k
 Wire Wire Line
@@
 Wire Wire Line
 	3700 3100 4850 3100
-Text Notes 4500 2100 0    50   ~ 0
-input\nvoltage +5 V
+Text Notes 5000 1900 0    50   ~ 0
+Vstup 5 V
 Text Notes 7500 2850 0    50   ~ 0
-output\nvoltage +5 V
+Výstup 5 V
 $Comp
 L Device:R R5
@@
 $EndComp
 $Comp
-L passive_components_rl:resisitor_variable_eu_rl R17
+L ochrana-napajeni-1-wire-rescue:resisitor_variable_eu_rl-passive_components_rl R17
 U 1 1 5FE1E7CE
 P 6100 3800

Commit message: Adding of HW parts and small changes.
Parts:
- C2: value 1,2n -> 1n2
- P3: value 1x2_pins_header_rl -> 1x2_pins_header
- R12: value 200 -> 200R
- R21: value 604 -> 604R
Connections:
- net at U1.8 (RTN): now also C2.2, R12.2, R18.2
- no-connect marks 0 -> 3
Other:
- note added: "max. I = 0,073 A\n114k64"
- note added: "Červená LED\nLTL-42NEW8D"
- note removed: "max. I = 0,073 A\n114,64k"
- note removed: "Červená LED"
Changed lines of the file:
@@
 P 6650 3850
 F 0 "C2" V 6604 3960 50  0000 L CNN
-F 1 "1,2n" V 6695 3960 50  0000 L CNN
+F 1 "1n2" V 6695 3960 50  0000 L CNN
 F 2 "capacitors_smd_rl:c_1206_rl" H 6650 3850 50  0001 C CNN
 F 3 "" H 6650 3850 50  0001 C CNN
@@
 P 7000 3500
 F 0 "P3" H 6750 3500 50  0000 L CNN
-F 1 "1x2_pins_header_rl" H 6600 3600 50  0000 L CNN
+F 1 "1x2_pins_header" H 6600 3600 50  0000 L CNN
 F 2 "Connector_PinHeader_2.54mm:PinHeader_1x02_P2.54mm_Vertical" H 7050 3500 50  0001 C CNN
 F 3 "" H 7050 3500 50  0001 C CNN
@@
 Wire Wire Line
 	7050 3300 7050 3350
-Text Notes 7000 3750 0    50   ~ 0
-Červená LED
+Text Notes 7000 3850 0    50   ~ 0
+Červená LED\nLTL-42NEW8D
 Wire Wire Line
 	6100 3400 6100 3650
@@
 	7100 2900 7450 2900
 Text Notes 5300 4250 0    50   ~ 0
-max. I = 0,073 A\n114,64k
+max. I = 0,073 A\n114k64
 Wire Wire Line
 	3700 3950 3700 4150
@@
 P 3700 4300
 F 0 "R12" H 3770 4346 50  0000 L CNN
-F 1 "200" H 3770 4255 50  0000 L CNN
+F 1 "200R" H 3770 4255 50  0000 L CNN
 F 2 "" V 3630 4300 50  0001 C CNN
 F 3 "~" H 3700 4300 50  0001 C CNN
@@
 P 7050 3150
 F 0 "R21" H 7120 3196 50  0000 L CNN
-F 1 "604" H 7120 3105 50  0000 L CNN
+F 1 "604R" H 7120 3105 50  0000 L CNN
 F 2 "" V 6980 3150 50  0001 C CNN
 F 3 "~" H 7050 3150 50  0001 C CNN
@@
 	0    1    1    0
 $EndComp
+NoConn ~ 5750 3500
+NoConn ~ 4850 3500
+NoConn ~ 4850 3400
 $EndSCHEMATC

Commit message: Changing of schematics.
Parts:
- removed P3: 1x2_pins_header, Connector_PinHeader_2.54mm:PinHeader_1x02_P2.54mm_Vertical, symbol ochrana-napajeni-1-wire-rescue:1x2_pins_header_rl-connectors_rl
- added D1: LTL-42NEW8D, symbol diode_rl:LED
Connections:
- net at U1.14 (FLT): now also D1.1 (K)
- net at U1.8 (RTN): now also C2.2, R12.2, R18.2
- net at R21.2: now also D1.2 (A)
Other:
- note removed: "Červená LED\nLTL-42NEW8D"
Changed lines of the file:
@@
 Connection ~ 7050 2900
-Wire Wire Line
-	6950 3350 6950 3100
-Wire Wire Line
-	6950 3100 5750 3100
-$Comp
-L ochrana-napajeni-1-wire-rescue:1x2_pins_header_rl-connectors_rl P3
-U 1 1 5F29F6AB
-P 7000 3500
-F 0 "P3" H 6750 3500 50  0000 L CNN
-F 1 "1x2_pins_header" H 6600 3600 50  0000 L CNN
-F 2 "Connector_PinHeader_2.54mm:PinHeader_1x02_P2.54mm_Vertical" H 7050 3500 50  0001 C CNN
-F 3 "" H 7050 3500 50  0001 C CNN
-	1    7000 3500
-	-1   0    0    1
-$EndComp
-Wire Wire Line
-	7050 3300 7050 3350
-Text Notes 7000 3850 0    50   ~ 0
-Červená LED\nLTL-42NEW8D
 Wire Wire Line
 	6100 3400 6100 3650
@@
 NoConn ~ 4850 3500
 NoConn ~ 4850 3400
+$Comp
+L diode_rl:LED D1
+U 1 1 619687DC
+P 7050 3500
+F 0 "D1" V 7050 3400 50  0000 C CNN
+F 1 "LTL-42NEW8D" V 6800 3200 50  0000 C CNN
+F 2 "" H 7050 3500 50  0001 C CNN
+F 3 "~" H 7050 3500 50  0001 C CNN
+	1    7050 3500
+	0    -1   -1   0
+$EndComp
+Wire Wire Line
+	7050 3300 7050 3350
+Wire Wire Line
+	7050 3650 7050 3700
+Wire Wire Line
+	7050 3700 6800 3700
+Wire Wire Line
+	6800 3700 6800 3100
+Wire Wire Line
+	5750 3100 6800 3100
 $EndSCHEMATC
