File: kicad/ochrany-1-wire/ochrany-1-wire.sch (KiCad schematic (older format))
At the start: 15 parts, among them P1 1x2_pins_header, P5 1x2_pins_header, P6 1x2_pins_header, P7 1x2_pins_header, P8 1x2_pins_header, Q1 BSS138P, Q4 BSS138P

Commit message: Adding of information and small changes. Remove main.pdf is too large.
Parts:
- D16, D7: value undir_transil -> ESD9L5.0ST5G
Changed lines of the file:
@@
 P 5150 2800
 F 0 "D7" H 5244 2846 50  0000 L CNN
-F 1 "undir_transil" H 5244 2755 50  0000 L CNN
+F 1 "ESD9L5.0ST5G" H 5244 2755 50  0000 L CNN
 F 2 "diodes_smd_rl:sod_923_rl" H 5150 2800 50  0001 C CNN
 F 3 "" H 5150 2800 50  0001 C CNN
@@
 P 5150 4400
 F 0 "D16" H 5244 4446 50  0000 L CNN
-F 1 "undir_transil" H 5244 4355 50  0000 L CNN
+F 1 "ESD9L5.0ST5G" H 5244 4355 50  0000 L CNN
 F 2 "diodes_smd_rl:sod_923_rl" H 5150 4400 50  0001 C CNN
 F 3 "" H 5150 4400 50  0001 C CNN
@@
 	5150 2950 5150 3000
 Wire Wire Line
-	5150 3000 5750 3000
-Wire Wire Line
-	5750 3000 5750 2700
-Wire Wire Line
-	5750 2700 5850 2700
+	5150 3000 5800 3000
+Wire Wire Line
+	5800 3000 5800 2700
+Wire Wire Line
+	5800 2700 5850 2700
 $Comp
 L esd_protection_1_wire_rpi-rescue:GND-power-esd_protection_1_wire_rpi-rescue #PWR016
@@
 	5150 4600 5150 4550
 Wire Wire Line
-	5150 4600 5750 4600
+	5150 4600 5800 4600
 $Comp
 L esd_protection_1_wire_rpi-rescue:GND-power-esd_protection_1_wire_rpi-rescue #PWR0131
@@
 	5150 4200 5850 4200
 Wire Wire Line
-	5750 4600 5750 4300
-Wire Wire Line
-	5750 4300 5850 4300
+	5800 4600 5800 4300
+Wire Wire Line
+	5800 4300 5850 4300
 Wire Wire Line
 	4900 2600 5150 2600

Commit message: Adding of new parts and modify old parts.
Parts:
- D15, D5: symbol diodes_rl:DS9503_eu_rl -> ochrany-1-wire-rescue:DS9503_eu_rl-diodes_rl
- P1, P5, P6, P7, P8: symbol connectors_rl:1x2_pins_header_rl -> ochrany-1-wire-rescue:1x2_pins_header_rl-connectors_rl
Other:
- note added: "Převodník log. úrovně"
- note removed: "level shifter"
Changed lines of the file:
@@
 $EndComp
 $Comp
-L connectors_rl:1x2_pins_header_rl P1
+L ochrany-1-wire-rescue:1x2_pins_header_rl-connectors_rl P1
 U 1 1 5E76B5E1
 P 3800 2650
@@
 	4300 3700 4300 3800
 $Comp
-L connectors_rl:1x2_pins_header_rl P5
+L ochrany-1-wire-rescue:1x2_pins_header_rl-connectors_rl P5
 U 1 1 5EE25312
 P 3800 4250
@@
 data_max31850k
 $Comp
-L connectors_rl:1x2_pins_header_rl P6
+L ochrany-1-wire-rescue:1x2_pins_header_rl-connectors_rl P6
 U 1 1 5EE4C5C1
 P 7000 3450
@@
 	7150 3500 7150 4200
 $Comp
-L connectors_rl:1x2_pins_header_rl P7
+L ochrany-1-wire-rescue:1x2_pins_header_rl-connectors_rl P7
 U 1 1 5F094A85
 P 6750 2450
@@
 	6800 2600 7150 2600
 $Comp
-L connectors_rl:1x2_pins_header_rl P8
+L ochrany-1-wire-rescue:1x2_pins_header_rl-connectors_rl P8
 U 1 1 5F0992AD
 P 6750 4350
@@
 	0    1    1    0
 $EndComp
-Text Notes 4350 3250 0    50   ~ 0
-level shifter
-$Comp
-L power_rl:+3,3V #PWR?
+Text Notes 4100 3200 0    50   ~ 0
+Převodník log. úrovně
+$Comp
+L ochrany-1-wire-rescue:+3,3V-power_rl #PWR?
 U 1 1 5FE0F44B
 P 4300 2000
@@
 $EndComp
 $Comp
-L power_rl:+3,3V #PWR?
+L ochrany-1-wire-rescue:+3,3V-power_rl #PWR?
 U 1 1 5FE0FC9F
 P 4300 3600
@@
 $EndComp
 $Comp
-L diodes_rl:DS9503_eu_rl D5
+L ochrany-1-wire-rescue:DS9503_eu_rl-diodes_rl D5
 U 1 1 5FE0BC8E
 P 6150 2700
@@
 $EndComp
 $Comp
-L diodes_rl:DS9503_eu_rl D15
+L ochrany-1-wire-rescue:DS9503_eu_rl-diodes_rl D15
 U 1 1 5FE0C859
 P 6150 4300

Commit message: Changing of schematics.
Other:
- note added: "Připojení k \ncentrální jednotce"
Changed lines of the file:
@@
 	1    0    0    -1
 $EndComp
+Text Notes 3600 2950 0    50   ~ 0
+Připojení k \ncentrální jednotce
+Text Notes 3600 4550 0    50   ~ 0
+Připojení k \ncentrální jednotce
 $EndSCHEMATC
