File: kicad/zonovy-regulator-mosfet-pwm-1-kanal/zonovy-regulator-mosfet-pwm-1-kanal.sch (KiCad schematic (older format))
At the start: 7 parts, among them J1 EBBA-02-C-SS-BU, Q1 DMN3023L-7, SW1 B144

Commit message: Adding of HW parts and small changes.
Parts:
- J1: value EBBA-02-C-SS-BU -> 1x2_screw_term_block
- R1: value 2,2k -> 2k2
Other:
- note added: "PE"
- note added: "Termoelektrický ventil"
- note added: "Zelená LED"
- note removed: "Zelená LED\nLTL-42NGY8D\nUf = 2 V\nIf = 10 mA"
Changed lines of the file:
@@
 P 11200 5600
 F 0 "J1" H 11280 5642 50  0000 L CNN
-F 1 "EBBA-02-C-SS-BU" H 11280 5551 50  0000 L CNN
+F 1 "1x2_screw_term_block" H 11280 5551 50  0000 L CNN
 F 2 "terminal_blocks_th_rl:xy301v_a_5_2p_rl" H 11200 5600 50  0001 C CNN
 F 3 "" H 11200 5600 50  0001 C CNN
@@
 P 12700 5950
 F 0 "R1" V 12654 6018 50  0000 L CNN
-F 1 "2,2k" V 12745 6018 50  0000 L CNN
+F 1 "2k2" V 12745 6018 50  0000 L CNN
 F 2 "resistors_smd_rl:r_1206_rl" H 12700 5950 50  0001 C CNN
 F 3 "" H 12700 5950 50  0001 C CNN
@@
 Wire Wire Line
 	10200 6050 10450 6050
-Text Notes 13100 6150 0    50   ~ 0
-Zelená LED\nLTL-42NGY8D\nUf = 2 V\nIf = 10 mA
+Text Notes 12950 6200 0    50   ~ 0
+Zelená LED
 Wire Wire Line
 	12700 6550 12400 6550
@@
 Pouzdro\npřepínače
 NoConn ~ 11900 5950
+Text Notes 12700 7150 0    50   ~ 0
+PE
+Text Notes 11400 5550 0    50   ~ 0
+Termoelektrický ventil
 $EndSCHEMATC

Commit message: Compress of image. Metadata for PDF information. Small changes.
Other:
- note added: "Termoelektrický pohon"
- note removed: "Termoelektrický ventil"
Changed lines of the file:
@@
 PE
 Text Notes 11400 5550 0    50   ~ 0
-Termoelektrický ventil
+Termoelektrický pohon
 $EndSCHEMATC
